File: hardware/dmx_controller.kicad_sch (KiCad schematic)
At the start: 1 part, among them T1 Screw_Terminal_01x02

Commit message: hardware update
Changed lines of the file:
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@@
 	(wire
 		(pts
-			(xy 190.5 67.31) (xy 203.2 67.31)
+			(xy 154.94 67.31) (xy 203.2 67.31)
 		)
 		(stroke
@@
 	(wire
 		(pts
-			(xy 190.5 69.85) (xy 203.2 69.85)
-		)
-		(stroke
-			(width 0)
-			(type default)
-		)
-	)
-	(wire
-		(pts
-			(xy 190.5 74.93) (xy 203.2 74.93)
-		)
-		(stroke
-			(width 0)
-			(type default)
-		)
-	)
-	(wire
-		(pts
-			(xy 190.5 72.39) (xy 203.2 72.39)
-		)
-		(stroke
-			(width 0)
-			(type default)
-		)
-	)
-	(wire
-		(pts
-			(xy 190.5 62.23) (xy 203.2 62.23)
-		)
-		(stroke
-			(width 0)
-			(type default)
-		)
-	)
-	(wire
-		(pts
-			(xy 190.5 64.77) (xy 203.2 64.77)
-		)
-		(stroke
-			(width 0)
-			(type default)
-		)
-	)
-	(wire
-		(pts
-			(xy 190.5 57.15) (xy 203.2 57.15)
+			(xy 154.94 69.85) (xy 203.2 69.85)
+		)
+		(stroke
+			(width 0)
+			(type default)
+		)
+	)
+	(wire
+		(pts
+			(xy 154.94 74.93) (xy 203.2 74.93)
+		)
+		(stroke
+			(width 0)
+			(type default)
+		)
+	)
+	(wire
+		(pts
+			(xy 154.94 72.39) (xy 203.2 72.39)
+		)
+		(stroke
+			(width 0)
+			(type default)
+		)
+	)
+	(wire
+		(pts
+			(xy 154.94 62.23) (xy 203.2 62.23)
+		)
+		(stroke
+			(width 0)
+			(type default)
+		)
+	)
+	(wire
+		(pts
+			(xy 154.94 64.77) (xy 203.2 64.77)
+		)
+		(stroke
+			(width 0)
+			(type default)
+		)
+	)
+	(wire
+		(pts
+			(xy 154.94 57.15) (xy 203.2 57.15)
 		)
 		(stroke
@@
 	(wire
 		(pts
-			(xy 190.5 59.69) (xy 203.2 59.69)
+			(xy 154.94 59.69) (xy 203.2 59.69)
 		)
 		(stroke
@@
 	)
 	(sheet
-		(at 160.02 50.8)
+		(at 124.46 50.8)
 		(size 30.48 26.67)
 		(exclude_from_sim no)
@@
 		)
 		(property "Sheetname" "analog_conditioning"
-			(at 160.02 50.0884 0)
+			(at 124.46 50.0884 0)
 			(effects
 				(font
@@
 		)
 		(property "Sheetfile" "analog_conditioning.kicad_sch"
-			(at 160.02 78.0546 0)
+			(at 124.46 78.0546 0)
 			(effects
 				(font
@@
 		)
 		(pin "adc3_5" output
-			(at 190.5 69.85 0)
+			(at 154.94 69.85 0)
 			(effects
 				(font
@@
 		)
 		(pin "adc3_6" output
-			(at 190.5 72.39 0)
+			(at 154.94 72.39 0)
 			(effects
 				(font
@@
 		)
 		(pin "adc3_2" output
-			(at 190.5 62.23 0)
+			(at 154.94 62.23 0)
 			(effects
 				(font
@@
 		)
 		(pin "adc3_0" output
-			(at 190.5 57.15 0)
+			(at 154.94 57.15 0)
 			(effects
 				(font
@@
 		)
 		(pin "adc3_1" output
-			(at 190.5 59.69 0)
+			(at 154.94 59.69 0)
 			(effects
 				(font
@@
 		)
 		(pin "adc3_3" output
-			(at 190.5 64.77 0)
+			(at 154.94 64.77 0)
 			(effects
 				(font
@@
 		)
 		(pin "adc3_7" output
-			(at 190.5 74.93 0)
+			(at 154.94 74.93 0)
 			(effects
 				(font
@@
 		)
 		(pin "adc3_4" output
-			(at 190.5 67.31 0)
-			(effects
-				(font
+			(at 154.94 67.31 0)
+			(effects
+				(font

Commit message: hardware update
Other:
- added sheet preamps (preamps.kicad_sch)
Changed lines of the file:
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@@
+	)
+	(sheet
+		(at 59.944 46.99)
+		(size 43.434 70.104)
+		(exclude_from_sim no)
+		(in_bom yes)
+		(on_board yes)
+		(dnp no)
+		(fields_autoplaced yes)
+		(stroke
+			(width 0.1524)
+			(type solid)
+		)
+		(fill
+			(color 0 0 0 0.0000)
+		)
+		(property "Sheetname" "preamps"
+			(at 59.944 46.2784 0)
+			(effects
+				(font
+					(size 1.27 1.27)
+				)
+				(justify left bottom)
+			)
+		)
+		(property "Sheetfile" "preamps.kicad_sch"
+			(at 59.944 117.6786 0)
+			(effects
+				(font
+					(size 1.27 1.27)
+				)
+				(justify left top)
+			)
+		)
+		(instances
+			(project "dmx_controller"
+				(path "/c888dd99-01b7-4b4b-82e5-501bcedd41ed"
+					(page "4")
+				)
+			)
+		)
 	)
 	(sheet
