File: hardware/mcu.kicad_sch (KiCad schematic)
At the start: 5 parts, among them CN10 Conn_02x17_Odd_Even, CN7 Conn_02x10_Odd_Even, CN8 Conn_02x08_Odd_Even, CN9 Conn_02x15_Odd_Even, U3 NUCLEO144-H743ZI

Commit message: hardware update
Changed lines of the file:
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@@
 	(wire
 		(pts
+			(xy 43.18 119.38) (xy 53.34 119.38)
+		)
+		(stroke
+			(width 0)
+			(type default)
+		)
+	)
+	(wire
+		(pts
 			(xy 66.04 91.44) (xy 76.2 91.44)
 		)
@@
 	(wire
 		(pts
-			(xy 21.59 119.38) (xy 53.34 119.38)
-		)
-		(stroke
-			(width 0)
-			(type default)
-		)
-	)
-	(wire
-		(pts
 			(xy 93.98 154.94) (xy 106.68 154.94)
 		)
@@
 		(effects
 			(font
-				(size 1.27 1.27)
-			)
-			(justify right)
-		)
-	)
-	(hierarchical_label "adc3_0"
-		(shape input)
-		(at 26.67 133.35 180)
-		(effects
-			(font
