File: hardware/dmx_controller.kicad_pcb (KiCad board)
At the start: 2 copper layers, 134.2 x 138.9 mm, 75 parts, among them CN10 Conn_02x17_Odd_Even, CN7 Conn_02x10_Odd_Even, CN8 Conn_02x08_Odd_Even, CN9 Conn_02x15_Odd_Even, J1 AudioJack2, J2 AudioJack2, J3 Conn_02x05_Odd_Even, J3 IDC 02x05, J4 Conn_02x05_Odd_Even, T1 Screw_Terminal_01x02, U1 TL072, U2 TL072, U201 MCP6002-xSN, U3 NUCLEO144-H743ZI

Commit message: hardware update
Parts:
- J1 (x2), J2 (x2): footprint Connector_Audio:Jack_6.35mm_Neutrik_NMJ6HFD2-AU_Horizontal -> light_controller:Cheap Jack
- moved T1 186.1 mm to (177.5, 63.4), turned to 180 degrees
- moved U3 141.0 mm to (204.7, 138.6), turned to 90 degrees
- moved CN7 118.7 mm to (205.7, 85.2), turned to -90 degrees
- moved CN8 115.7 mm to (214.8, 131.0), turned to 90 degrees
- moved R203 105.1 mm to (212.6, 113.2), turned to 180 degrees
- moved C203 104.2 mm to (212.6, 111.2), turned to 0 degrees
- moved R204 103.3 mm to (212.6, 109.2), turned to 0 degrees
- moved C204 102.7 mm to (212.6, 107.2), turned to 180 degrees
- moved U201 92.7 mm to (218.2, 110.2), turned to 180 degrees
- moved R201 83.3 mm to (224.0, 113.0), turned to 0 degrees
- moved C201 82.1 mm to (223.9, 111.0), turned to 180 degrees
- moved CN9 81.3 mm to (237.7, 131.0), turned to -90 degrees
- moved R202 81.1 mm to (223.9, 109.0), turned to 180 degrees
- moved C202 80.2 mm to (223.9, 107.0), turned to 0 degrees
- moved CN10 67.6 mm to (232.6, 85.2), turned to -90 degrees
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Routing:
- net Net-(J3-Pin_7): track 26.9 -> 27.8 mm
Other:
- board size 134.2 x 138.9 mm -> 181.3 x 136.9 mm

Commit message: hardware update
Parts:
- removed the C1 at (304.2, 174.3)
- removed the C10 at (309.3, 171.0)
- removed the C11 at (306.4, 174.3)
- removed the C12 at (285.5, 174.3)
- removed the C2 at (306.2, 185.7)
- removed the C3 at (307.3, 163.9)
- removed the C4 at (283.5, 174.3)
- removed the C5 at (285.8, 185.7)
- removed the C6 at (275.5, 163.9)
- removed the C7 at (273.7, 170.9)
- removed the C8 at (302.1, 185.7)
- removed the C9 at (281.7, 185.7)
- removed the D1 at (297.2, 178.2)
- removed the D2 at (299.2, 178.2)
- removed the D3 at (278.3, 178.3)
- removed the D4 at (276.3, 178.3)
- removed the J1 at (310.2, 178.6)
- removed the J2 at (289.2, 178.6)
- removed the J3 at (296.8, 163.9)
- removed the R1 at (298.1, 174.3)
- removed the R2 at (304.2, 185.7)
- removed the R3 at (302.1, 174.3)
- removed the R4 at (300.1, 174.3)
- removed the R5 at (277.4, 174.3)
- removed the R6 at (283.7, 185.7)
- removed the R7 at (281.5, 174.3)
- removed the R8 at (279.4, 174.3)
- removed the U1 at (304.6, 180.0)
- removed the U2 at (283.6, 180.0)
- added C205: 5n6, Capacitor_SMD:C_0805_2012Metric, F.Cu at (320.6, 119.0)
- added C206: 3n3, Capacitor_SMD:C_0805_2012Metric, F.Cu at (320.6, 122.0)
- added J202: Conn_02x05_Odd_Even, Connector_IDC:IDC-Header_2x05_P2.54mm_Vertical, F.Cu at (339.4, 93.1)
- added R203: 10k, Resistor_SMD:R_0805_2012Metric, F.Cu at (355.7, 122.4)
- added R204: 10k, Resistor_SMD:R_0805_2012Metric, F.Cu at (355.7, 125.3)
- added R205: 10k, Resistor_SMD:R_0805_2012Metric, F.Cu at (355.7, 128.3)
- added R206: 10k, Resistor_SMD:R_0805_2012Metric, F.Cu at (355.7, 131.2)
- added R207: 10k, Resistor_SMD:R_0805_2012Metric, F.Cu at (355.7, 134.2)
- added R210: 10k, Resistor_SMD:R_0805_2012Metric, F.Cu at (360.1, 122.4)
- added R211: 10k, Resistor_SMD:R_0805_2012Metric, F.Cu at (360.1, 125.3)
- added R212: 10k, Resistor_SMD:R_0805_2012Metric, F.Cu at (360.1, 128.3)
- added R213: 2k61, Resistor_SMD:R_0805_2012Metric, F.Cu at (325.0, 118.9)
- added R214: 7k15, Resistor_SMD:R_0805_2012Metric, F.Cu at (325.0, 121.8)
- added U201: TL072, Package_SO:SOIC-8_3.9x4.9mm_P1.27mm, F.Cu at (331.5, 114.9)
- added U202: TL072, Package_SO:SOIC-8_3.9x4.9mm_P1.27mm, F.Cu at (333.9, 143.5)
- J201: renamed from J4; moved to F.Cu
- moved T1 203.1 mm to (370.5, 126.8), turned to 0 degrees
- moved C2 140.0 mm to (369.2, 47.1), turned to 180 degrees
- moved R2 138.3 mm to (369.2, 49.1), turned to 180 degrees
- moved C8 136.7 mm to (369.2, 51.2), turned to 180 degrees
- moved J1 135.8 mm to (362.1, 43.1), turned to 0 degrees
- moved U1 132.2 mm to (363.5, 48.8), turned to 0 degrees
- moved C11 127.6 mm to (357.8, 47.0), turned to 180 degrees
- moved C10 127.0 mm to (354.5, 44.0), turned to 0 degrees
- moved R208 126.4 mm to (333.5, 149.9), turned to -90 degrees
- moved D2 125.6 mm to (361.7, 54.1), turned to 180 degrees
- moved C1 125.6 mm to (357.8, 49.1), turned to 0 degrees
- moved C5 125.0 mm to (369.2, 67.6), turned to 180 degrees
- moved D1 124.0 mm to (361.7, 56.1), turned to 180 degrees
- moved R6 123.8 mm to (369.2, 69.6), turned to 180 degrees
- moved R3 123.8 mm to (357.8, 51.2), turned to 0 degrees
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- renumbered R203 to R208, R204 to R209, U201 to U203
Connections:
- C201 pad 2: adc3_0 -> Net-(U201B--)
- C202 pad 1: Net-(U201A-+) -> Net-(U201B-+)
- C203 pad 2: adc3_1 -> Net-(U202B--)
- C204 pad 1: Net-(U201B-+) -> Net-(U202B-+)
- J3 pad 3: Net-(U1B--) -> Net-(J3-Pin_3)
- J3 pad 4: (no net) -> Net-(J3-Pin_3)
- J3 pad 7: Net-(U2B--) -> Net-(J3-Pin_7)
- J3 pad 8: (no net) -> Net-(J3-Pin_7)
- R201 pad 1: /analog_conditioning/analog_in_1 -> Net-(U201A--)
- R202 pad 2: Net-(U201A-+) -> Net-(U201B-+)
- R208 pad 1: /analog_conditioning/analog_in_2 -> Net-(U202A--)
- R209 pad 2: Net-(U201B-+) -> Net-(U202B-+)
- U1 pad 6: Net-(U1B--) -> Net-(J3-Pin_3)
- U1 pad 7: Net-(U1B--) -> Net-(J3-Pin_3)
- U2 pad 6: Net-(U2B--) -> Net-(J3-Pin_7)
- U2 pad 7: Net-(U2B--) -> Net-(J3-Pin_7)
- U203 pad 1: adc3_0 -> /analog_conditioning/analog_out_1
- U203 pad 2: adc3_0 -> Net-(U203A--)
- U203 pad 3: Net-(U201A-+) -> Net-(U203A-+)
- U203 pad 5: Net-(U201B-+) -> Net-(U203B-+)
- U203 pad 6: adc3_1 -> Net-(U203B--)
- U203 pad 7: adc3_1 -> /analog_conditioning/analog_out_2
Routing:
- net GND: track 364.0 -> 190.6 mm, vias 24 -> 12
- net +12V: track 121.6 -> 60.8 mm, vias 4 -> 2
- net -12V: track 103.5 -> 51.7 mm, vias 4 -> 2
- net Net-(U1B--): track 27.6 -> 0.00 mm
- net Net-(U2B--): track 26.9 -> 0.00 mm
- net Net-(D1-K): track 53.0 -> 26.5 mm
- net Net-(D3-K): track 46.1 -> 23.1 mm
- net Net-(D3-A): track 36.6 -> 18.3 mm
- net Net-(D1-A): track 30.0 -> 15.0 mm
- net Net-(C3-Pad2): track 26.8 -> 13.4 mm, vias 2 -> 1
- net Net-(C6-Pad2): track 26.8 -> 13.4 mm, vias 2 -> 1
- net Net-(C3-Pad1): track 26.5 -> 13.2 mm, vias 2 -> 1
- net Net-(C6-Pad1): track 21.6 -> 10.8 mm, vias 2 -> 1
- net Net-(C1-Pad1): track 18.9 -> 9.45 mm
- net Net-(C4-Pad1): track 18.3 -> 8.96 mm
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Other:
- board size 181.3 x 136.9 mm -> 170.2 x 114.9 mm

Commit message: analog conditioning and preamp board sent for prototype manufacture
Parts:
- removed CN10: Conn_02x17_Odd_Even, Connector_PinSocket_2.54mm:PinSocket_2x17_P2.54mm_Vertical
- removed CN7: Conn_02x10_Odd_Even, Connector_PinSocket_2.54mm:PinSocket_2x10_P2.54mm_Vertical
- removed CN8: Conn_02x08_Odd_Even, Connector_PinHeader_2.54mm:PinHeader_2x08_P2.54mm_Vertical
- removed CN9: Conn_02x15_Odd_Even, Connector_PinSocket_2.54mm:PinSocket_2x15_P2.54mm_Vertical
- added C207: 3n3, Capacitor_SMD:C_0805_2012Metric, B.Cu at (422.4, 59.2)
- added C208: 3n3, Capacitor_SMD:C_0805_2012Metric, B.Cu at (422.4, 61.2)
- added C209: 100n, Capacitor_SMD:C_0805_2012Metric, B.Cu at (422.4, 29.0)
- added C210: 100n, Capacitor_SMD:C_0805_2012Metric, B.Cu at (434.4, 32.5)
- added C211: 100n, Capacitor_SMD:C_0805_2012Metric, B.Cu at (422.4, 53.2)
- added C212: 100n, Capacitor_SMD:C_0805_2012Metric, B.Cu at (434.1, 57.8)
- added C213: 100n, Capacitor_SMD:C_0805_2012Metric, B.Cu at (430.7, 49.0)
- added J203: Conn_01x10, Connector_PinHeader_2.54mm:PinHeader_1x10_P2.54mm_Vertical, F.Cu at (417.8, 64.0)
- added J204: Conn_01x10, Connector_PinHeader_2.54mm:PinHeader_1x10_P2.54mm_Vertical, F.Cu at (417.8, 25.9)
- added R215: 10k, Resistor_SMD:R_0805_2012Metric, B.Cu at (435.4, 50.9)
- added R216: 10k, Resistor_SMD:R_0805_2012Metric, B.Cu at (439.3, 50.9)
- added R217: 0R, Resistor_SMD:R_0805_2012Metric, B.Cu at (443.5, 35.4)
- added R218: 0R, Resistor_SMD:R_0805_2012Metric, B.Cu at (445.5, 35.4)
- added R219: 0R, Resistor_SMD:R_0805_2012Metric, B.Cu at (443.2, 54.9)
- added R220: 0R, Resistor_SMD:R_0805_2012Metric, B.Cu at (445.3, 54.9)
- added R221: 0R, Resistor_SMD:R_0805_2012Metric, B.Cu at (434.4, 30.5)
- added R222: 0R, Resistor_SMD:R_0805_2012Metric, B.Cu at (434.4, 28.5)
- added R223: 0R, Resistor_SMD:R_0805_2012Metric, B.Cu at (434.1, 53.8)
- added R224: 0R, Resistor_SMD:R_0805_2012Metric, B.Cu at (434.1, 55.8)
- added RV201: R_Potentiometer, Potentiometer_THT:Potentiometer_Bourns_3296W_Vertical, F.Cu at (443.8, 31.0)
- added RV202: R_Potentiometer, Potentiometer_THT:Potentiometer_Bourns_3296W_Vertical, F.Cu at (443.9, 59.3)
- C11, C12, C8, C9: value 220n -> 100n
- C201, C204, C205, R201, R202, R203, R206, R207, R212, R213, R214, U201, U202, U203: moved to B.Cu
- C202, C206: value 3n3 -> 5n6; moved to B.Cu
- C203: value 5n6 -> 3n3; moved to B.Cu
- R204, R210: value 10k -> 2k61; moved to B.Cu
- R205, R211: value 10k -> 7k15; moved to B.Cu
- R208: value 2k61 -> 10k; moved to B.Cu
- R209: value 7k15 -> 10k; moved to B.Cu
- moved R208 152.3 mm to (438.6, 39.6)
- moved C203 132.3 mm to (422.4, 35.0), turned to 180 degrees
- moved C202 131.4 mm to (422.4, 33.0)
- moved C201 130.7 mm to (422.4, 31.0), turned to 0 degrees
- moved R202 130.3 mm to (427.8, 35.7), turned to 90 degrees
- moved R201 130.1 mm to (429.8, 35.7), turned to -90 degrees
- moved U203 130.0 mm to (435.7, 45.2), turned to -90 degrees
- moved R209 130.0 mm to (430.6, 45.0)
- moved U202 129.0 mm to (428.4, 55.8), turned to 180 degrees
- moved U201 128.6 mm to (428.5, 30.4), turned to 180 degrees
- moved C204 128.0 mm to (422.4, 37.0)
- moved J201 123.9 mm to (445.3, 40.1), turned to 0 degrees
- moved R207 123.5 mm to (435.1, 39.6), turned to 90 degrees
- moved R213 121.8 mm to (432.0, 60.7), turned to 90 degrees
- moved C206 120.7 mm to (422.4, 57.2), turned to 180 degrees
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Connections:
- C202 pad 1: Net-(U201B-+) -> Net-(C201-Pad1)
- C202 pad 2: GND -> Net-(U201B--)
- C203 pad 1: Net-(C203-Pad1) -> Net-(U201B-+)
- C203 pad 2: Net-(U202B--) -> GND
- C204 pad 1: Net-(U202B-+) -> Net-(U201B-+)
- C205 pad 1: Net-(C201-Pad1) -> Net-(C205-Pad1)
- C205 pad 2: Net-(U201B--) -> Net-(U202B--)
- C206 pad 1: Net-(U201B-+) -> Net-(C205-Pad1)
- C206 pad 2: GND -> Net-(U202B--)
- R201 pad 1: Net-(U201A--) -> Net-(R201-Pad1)
- R204 pad 1: Net-(U203A-+) -> Net-(R201-Pad1)
- R204 pad 2: /analog_conditioning/V_REF_1_65V -> Net-(C201-Pad1)
- R205 pad 1: /analog_conditioning/analog_out_1 -> Net-(C201-Pad1)
- R205 pad 2: Net-(U203A--) -> Net-(U201B-+)
- R206 pad 1: Net-(U203A--) -> Net-(U203A-+)
- R206 pad 2: GND -> /analog_conditioning/V_REF_1_65V
- R207 pad 1: /analog_conditioning/V_REF_1_65V -> /analog_conditioning/analog_out_1
- R207 pad 2: Net-(U203B-+) -> Net-(U203A--)
- R208 pad 1: Net-(U202A--) -> Net-(U203A--)
- R208 pad 2: Net-(C203-Pad1) -> GND
- R209 pad 1: Net-(C203-Pad1) -> /analog_conditioning/V_REF_1_65V
- R209 pad 2: Net-(U202B-+) -> Net-(U203B-+)
- R210 pad 1: Net-(U202B--) -> Net-(R210-Pad1)
- R210 pad 2: Net-(U203B-+) -> Net-(C205-Pad1)
- R211 pad 1: /analog_conditioning/analog_out_2 -> Net-(C205-Pad1)
- R211 pad 2: Net-(U203B--) -> Net-(U202B-+)
- R212 pad 1: Net-(U203B--) -> Net-(U202B--)
- R212 pad 2: GND -> Net-(U203B-+)
- R213 pad 1: Net-(U201A--) -> Net-(R210-Pad1)
- R213 pad 2: Net-(C201-Pad1) -> Net-(C205-Pad1)
- R214 pad 1: Net-(C201-Pad1) -> Net-(C205-Pad1)
- R214 pad 2: Net-(U201B-+) -> Net-(U202B-+)
- U201 pad 1: Net-(U201A--) -> Net-(R201-Pad1)
- U201 pad 4: unconnected-(U201C-V--Pad4) -> -12V
- U201 pad 8: unconnected-(U201C-V+-Pad8) -> +12V
- U202 pad 1: Net-(U202A--) -> Net-(R210-Pad1)
- U202 pad 4: unconnected-(U202C-V--Pad4) -> -12V
- U202 pad 8: unconnected-(U202C-V+-Pad8) -> +12V
- U203 pad 6: Net-(U203B--) -> Net-(U203B-+)
Routing:
- net +12V: track 60.8 -> 171.8 mm, vias 2 -> 6
- net GND: track 190.6 -> 260.0 mm, vias 12 -> 22
- net /analog_conditioning/analog_out_1: track 0.00 -> 68.5 mm
- net /analog_conditioning/analog_out_2: track 0.00 -> 67.6 mm, vias 0 -> 6
- net +3.3V: track 0.00 -> 65.6 mm, vias 0 -> 5
- net -12V: track 51.7 -> 116.6 mm, vias 2 -> 4
- net /analog_conditioning/V_REF_1_65V: track 0.00 -> 60.7 mm, vias 0 -> 1
- net Net-(U201A-+): track 0.00 -> 23.9 mm
- net Net-(U202A-+): track 0.00 -> 21.3 mm
- net Net-(U202B--): track 0.00 -> 19.6 mm, vias 0 -> 4
- net Net-(U203B-+): track 0.00 -> 19.4 mm
- net Net-(U201B--): track 0.00 -> 17.6 mm, vias 0 -> 2
- net Net-(C201-Pad1): track 4.01 -> 17.1 mm
- net Net-(C205-Pad1): track 0.00 -> 11.7 mm
- net Net-(U202B-+): track 0.00 -> 9.77 mm, vias 0 -> 2
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Other:
- board size 170.2 x 114.9 mm -> 288.9 x 131.7 mm

Commit message: change?
Parts:
- added J203: Conn_01x10, Connector_PinHeader_2.54mm:PinHeader_1x10_P2.54mm_Vertical, B.Cu at (234.0, 107.4)
- added J203: Conn_01x10, Connector_PinHeader_2.54mm:PinHeader_1x10_P2.54mm_Vertical, B.Cu at (234.0, 64.7)
- added J203: Conn_01x10, Connector_PinHeader_2.54mm:PinHeader_1x10_P2.54mm_Vertical, B.Cu at (270.4, 107.4)
- added J203: Conn_01x10, Connector_PinHeader_2.54mm:PinHeader_1x10_P2.54mm_Vertical, B.Cu at (270.4, 64.7)
- added J204: Conn_01x10, Connector_PinHeader_2.54mm:PinHeader_1x10_P2.54mm_Vertical, B.Cu at (270.4, 102.8)
- added J204: Conn_01x10, Connector_PinHeader_2.54mm:PinHeader_1x10_P2.54mm_Vertical, B.Cu at (234.0, 102.8)
- added J204: Conn_01x10, Connector_PinHeader_2.54mm:PinHeader_1x10_P2.54mm_Vertical, B.Cu at (234.0, 145.5)
- added J204: Conn_01x10, Connector_PinHeader_2.54mm:PinHeader_1x10_P2.54mm_Vertical, B.Cu at (270.4, 145.5)
Routing:
- net /analog_conditioning/V_REF_1_65V: track 60.7 -> 61.6 mm
